Commit message: update bluerov2 package to work with latest uuv sim
update bluerov2 package to work with latest uuv sim

File: bluerov2_description/robots/bluerov2_default.xacro (robot description, xacro)
@@ -7,10 +7,11 @@
   <!-- Hydrodynamic and hydrostatic parameters for the vehicle xacro:macro bluerov2_hydro_model -->
   <xacro:include filename="$(find bluerov2_description)/urdf/gazebo.xacro"/>
-<!-- Create the bluerov2 -->
-  <xacro:bluerov2_base namespace="$(arg namespace)">
+  <!-- Create the bluerov2 -->
+  <xacro:bluerov2_base
+          namespace="$(arg namespace)">
     <!-- The underwater object plugin is given as an input block parameter to
      allow the addition of external models of manipulator units -->
     <gazebo>
-      <plugin name="uuv_plugin" filename="libunderwater_object_ros_plugin.so">
+      <plugin name="uuv_plugin" filename="libuuv_underwater_object_ros_plugin.so">
         <fluid_density>1028.0</fluid_density>
         <flow_velocity_topic>hydrodynamics/current_velocity</flow_velocity_topic>

File: bluerov2_description/urdf/base.xacro (robot description, xacro)
@@ -2,5 +2,5 @@
 <robot xmlns:xacro="http://www.ros.org/wiki/xacro">
   <!-- Loading some constants -->
-  <xacro:include filename="$(find uuv_descriptions)/models/common/urdf/common.urdf.xacro"/>
+  <xacro:include filename="$(find uuv_descriptions)/urdf/common.urdf.xacro"/>
   <!-- Loading file with sensor macros -->
   <xacro:include filename="$(find uuv_sensor_ros_plugins)/urdf/sensor_snippets.xacro"/>
@@ -45,38 +45,38 @@
   <!-- <xacro:macro name="bluerov2_base" params="namespace debug *gazebo"> -->
   <xacro:macro name="bluerov2_base" params="namespace *gazebo">
-      <!-- Rigid body description of the base link -->
-      <link name="${namespace}/base_link">
-        <!--
-          Be careful to setup the coefficients for the inertial tensor,
-          otherwise your model will become unstable on Gazebo
-        -->
-        <inertial>
-          <mass value="${mass}" />
-          <origin xyz="${cog}" rpy="0 0 0"/>
-          <!-- <inertia ixx="525.39" ixy="1.44" ixz="33.41" iyy="794.20" iyz="2.6" izz="691.23"/> -->
-          <inertia
-            ixx="${0.2*mass*y_size*y_size + 0.2*mass*z_size*z_size}" ixy="0.0" ixz="0.0"
-            iyy="${0.2*mass*x_size*x_size + 0.2*mass*z_size*z_size}" iyz="0.0"
-            izz="${0.2*mass*x_size*x_size + 0.2*mass*y_size*y_size}" />
-        </inertial>
-        <!-- This visual geometry representation can be used when running
-             tasks in which you need Gazebo to start quickly
-        -->
-        <!-- <xacro:if value="${use_simplified_mesh}"> -->
-        <!-- Code in rexrov2_base.xacro if use the flag use_simplified_mesh -->
-        <visual>
-          <origin xyz="0 0 0" rpy="0 0 0"/>
-          <geometry>
-            <mesh filename="${visual_mesh_file}" scale="1 1 1" />
-          </geometry>
-        </visual>
-        <!-- In rexrov2_base they made collision planes to minize the GPU load -->
-        <!-- <collision>
-          <origin xyz="0 0 0" rpy="0 0 0"/>
-          <geometry>
-            <mesh filename="${collision_mesh_file}" scale="1 1 1" />
-          </geometry>
-        </collision> -->
-      </link>
+    <!-- Rigid body description of the base link -->
+    <link name="${namespace}/base_link">
+      <!--
+        Be careful to setup the coefficients for the inertial tensor,
+        otherwise your model will become unstable on Gazebo
+      -->
+      <inertial>
+        <mass value="${mass}" />
+        <origin xyz="${cog}" rpy="0 0 0"/>
+        <!-- <inertia ixx="525.39" ixy="1.44" ixz="33.41" iyy="794.20" iyz="2.6" izz="691.23"/> -->
+        <inertia
+                ixx="${0.2*mass*y_size*y_size + 0.2*mass*z_size*z_size}" ixy="0.0" ixz="0.0"
+                iyy="${0.2*mass*x_size*x_size + 0.2*mass*z_size*z_size}" iyz="0.0"
+                izz="${0.2*mass*x_size*x_size + 0.2*mass*y_size*y_size}" />
+      </inertial>
+      <!-- This visual geometry representation can be used when running
+           tasks in which you need Gazebo to start quickly
+      -->
+      <!-- <xacro:if value="${use_simplified_mesh}"> -->
+      <!-- Code in rexrov2_base.xacro if use the flag use_simplified_mesh -->
+      <visual>
+        <origin xyz="0 0 0" rpy="0 0 0"/>
+        <geometry>
+          <mesh filename="${visual_mesh_file}" scale="1 1 1" />
+        </geometry>
+      </visual>
+      <!-- In rexrov2_base they made collision planes to minize the GPU load -->
+      <!-- <collision>
+        <origin xyz="0 0 0" rpy="0 0 0"/>
+        <geometry>
+          <mesh filename="${collision_mesh_file}" scale="1 1 1" />
+        </geometry>
+      </collision> -->
+    </link>
     <gazebo reference="${namespace}/base_link">
       <selfCollide>false</selfCollide>

File: bluerov2_description/urdf/sensors.xacro (robot description, xacro)
@@ -17,8 +17,8 @@
     <origin xyz="0 0 0" rpy="0 0 0"/>
   </xacro:default_pressure>
-  <!-- Beacon Sensor  -->
+  <!-- Beacon Sensor
   <xacro:default_beacon namespace="${namespace}" parent_link="${namespace}/base_link">
     <origin xyz="0 0 0" rpy="0 0 0"/>
-  </xacro:default_beacon>
+  </xacro:default_beacon>-->
   <!-- Mount a camera -->
   <!-- <xacro:default_camera namespace="${namespace}" parent_link="${namespace}/base_link" suffix="front">

File: bluerov2_description/urdf/snippets.xacro (robot description, xacro)
@@ -26,6 +26,6 @@
         <origin xyz="0 0 0" rpy="0 0 0"/>
         <inertia ixx="0.000000017" ixy="0.0" ixz="0.0"
-               iyy="0.000000017" iyz="0.0"
-               izz="0.000000017" />
+                 iyy="0.000000017" iyz="0.0"
+                 izz="0.000000017" />
       </inertial>
     </link>
@@ -40,44 +40,44 @@
     <gazebo>
       <!-- Thruster ROS plugin -->
-     <plugin name="${robot_namespace}_${thruster_id}_thruster_model" filename="libthruster_ros_plugin.so">
-       <!-- Name of the thruster link -->
-       <linkName>${robot_namespace}/thruster_${thruster_id}</linkName>
-       <!-- Name of the joint between thruster and vehicle base link -->
-       <jointName>${robot_namespace}/thruster_${thruster_id}_joint</jointName>
-       <!-- Make the thruster aware of its id -->
-       <thrusterID>${thruster_id}</thrusterID>
-       <!-- Gain of the input command signal -->
-       <gain>1</gain>
-       <!-- Maximum allowed input value for the input signal for thruster unit -->
-       <!-- <clampMax>0</clampMax> -->
-       <!-- Minimum allowed value for the input signal for thruster unit -->
-       <!-- <clampMin>0</clampMin> -->
-       <!-- Minimum and maximum thrust force output allowed -->
-       <!-- <thrustMin>0</thrustMin> -->
-       <!-- <thrustMax>200</thrustMax> -->
-       <!--
-       Value from 0 to 1 to set the efficiency of the output thrust force
-       Default value is 1.0
-       -->
-       <thrust_efficiency>1</thrust_efficiency>
-       <!--
-       Value from 0 to 1 to set the efficiency of the propeller as a factor
-       to be multiplied to the current value of the state variable at each
-       iteration.
-       Default value is 1.0
-       -->
-       <propeller_efficiency>1</propeller_efficiency>
-       <!-- 2) First order model -->
-       <dynamics>
-         <type>FirstOrder</type>
-         <timeConstant>0.2</timeConstant>
-       </dynamics>
-       <conversion>
-         <type>Basic</type>
-         <rotorConstant>0.00001</rotorConstant>
-         <!-- <rotorConstant>0</rotorConstant> -->
-       </conversion>
-     </plugin>
-   </gazebo>
+      <plugin name="${robot_namespace}_${thruster_id}_thruster_model" filename="libuuv_thruster_ros_plugin.so">
+        <!-- Name of the thruster link -->
+        <linkName>${robot_namespace}/thruster_${thruster_id}</linkName>
+        <!-- Name of the joint between thruster and vehicle base link -->
+        <jointName>${robot_namespace}/thruster_${thruster_id}_joint</jointName>
+        <!-- Make the thruster aware of its id -->
+        <thrusterID>${thruster_id}</thrusterID>
+        <!-- Gain of the input command signal -->
+        <gain>1</gain>
+        <!-- Maximum allowed input value for the input signal for thruster unit -->
+        <!-- <clampMax>0</clampMax> -->
+        <!-- Minimum allowed value for the input signal for thruster unit -->
+        <!-- <clampMin>0</clampMin> -->
+        <!-- Minimum and maximum thrust force output allowed -->
+        <!-- <thrustMin>0</thrustMin> -->
+        <!-- <thrustMax>200</thrustMax> -->
+        <!--
+        Value from 0 to 1 to set the efficiency of the output thrust force
+        Default value is 1.0
+        -->
+        <thrust_efficiency>1</thrust_efficiency>
+        <!--
+        Value from 0 to 1 to set the efficiency of the propeller as a factor
+        to be multiplied to the current value of the state variable at each
+        iteration.
+        Default value is 1.0
+        -->
+        <propeller_efficiency>1</propeller_efficiency>
+        <!-- 2) First order model -->
+        <dynamics>
+          <type>FirstOrder</type>
+          <timeConstant>0.2</timeConstant>
+        </dynamics>
+        <conversion>
+          <type>Basic</type>
+          <rotorConstant>0.00001</rotorConstant>
+          <!-- <rotorConstant>0</rotorConstant> -->
+        </conversion>
+      </plugin>
+    </gazebo>
     <gazebo reference="${robot_namespace}/thruster_${thruster_id}">
       <selfCollide>false</selfCollide>
