Commit message: started to add cpc sensor
started to add cpc sensor

File: bluerov2_description/urdf/sensors.xacro (robot description, xacro)
@@ -25,3 +25,9 @@
     <origin xyz="0 0 0.2" rpy="0 0 0"/>
   </xacro:default_camera> -->
+  <xacro:default_chemical_concentration_sensor_macro
+          namespace="${namespace}"
+          parent_link="${namespace}/base_link"
+          inertial_reference_frame="${inertial_reference_frame}">
+    <origin xyz="0 0 0" rpy="0 0 0"/>
+  </xacro:default_chemical_concentration_sensor_macro>
 </robot>
